File: hardware/SimpleFlightController.kicad_pcb (KiCad board)
At the start: 2 copper layers, 40 x 46 mm, 79 parts, among them J1 Screw_Terminal_01x02, J2 Conn_01x03, J3 Conn_01x03, U1 BQ25883RGER, U2 ICM-45686, U3 STM32F722RETx, U4 BMP580, U5 TPS63070RNMR, U6 LMR51430, X1 X322525MOB4SI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

Commit message: update image paths and 3d render
Routing:
- net GND: vias 6 -> 8
Changed lines of the file:
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@@
 					(face "Blender Pro Bold")
 					(size 0.5 0.5)
-					(thickness 0.15)
+					(thickness 0.125)
 				)
 			)
@@
 		)
 		(embedded_fonts no)
-		(model "/hardware/lib/lcsc.3dshapes/CRYSTAL-SMD_4P-L3.2-W2.5-BL.wrl"
+		(model "${KIPRJMOD}/lib/lcsc.3dshapes/CRYSTAL-SMD_4P-L3.2-W2.5-BL.step"
 			(offset
 				(xyz 0 -0 -0)
@@
 					(face "Blender Pro Bold")
 					(size 0.5 0.5)
-					(thickness 0.15)
+					(thickness 0.125)
 				)
 			)
@@
 		)
 		(embedded_fonts no)
-		(model "/hardware/lib/lcsc.3dshapes/USB-C-SMD_TYPE-C-6PIN-2MD-073.wrl"
+		(model "${KIPRJMOD}/lib/lcsc.3dshapes/USB-C-SMD_TYPE-C-6PIN-2MD-073.step"
 			(offset
-				(xyz 0 -1.2 0.9)
+				(xyz 0 -1.2 1.4)
 			)
 			(scale
@@
 			)
 			(rotate
-				(xyz 0 0 0)
+				(xyz -0 -0 -0)
 			)
 		)
@@
 					(face "Blender Pro Bold")
 					(size 0.5 0.5)
-					(thickness 0.15)
+					(thickness 0.125)
 				)
 			)
@@
 		)
 		(embedded_fonts no)
-		(model "/hardware/lib/lcsc.3dshapes/VFQFPN-24_L4.0-W4.0-H0.9-P0.50.wrl"
+		(model "${KIPRJMOD}/lib/lcsc.3dshapes/VFQFPN-24_L4.0-W4.0-H0.9-P0.50.step"
 			(offset
 				(xyz 0 -0 -0)
@@
 					(face "Blender Pro Bold")
 					(size 0.5 0.5)
-					(thickness 0.15)
+					(thickness 0.125)
 				)
 			)
@@
 		)
 		(embedded_fonts no)
-		(model "/hardware/lib/lcsc.3dshapes/LGA-14_L2.5-W3.0-H0.9-P0.50.wrl"
+		(model "${KIPRJMOD}/lib/lcsc.3dshapes/LGA-14_L2.5-W3.0-H0.9-P0.50.step"
 			(offset
-				(xyz 0.24 -0.37 -0)
+				(xyz 0 0 -0)
 			)
 			(scale
@@
 			)
 			(rotate
-				(xyz 0 0 0)
+				(xyz -0 -0 -0)
 			)
 		)
@@
 					(face "Blender Pro Bold")
 					(size 0.5 0.5)
-					(thickness 0.15)
+					(thickness 0.125)
 				)
 			)
@@
 		)
 		(embedded_fonts no)
-		(model "/hardware/lib/lcsc.3dshapes/IND-SMD_L3.0-W3.0-H1.5.wrl"
+		(model "${KIPRJMOD}/lib/lcsc.3dshapes/IND-SMD_L3.0-W3.0-H1.5.step"
 			(offset
 				(xyz 0 -0 -0)
@@
 					(face "Blender Pro Bold")
 					(size 0.5 0.5)
-					(thickness 0.15)
+					(thickness 0.125)
 				)
 			)
@@
 		)
 		(embedded_fonts no)
-		(model "/hardware/lib/lcsc.3dshapes/VQFN-HR-15_L3.0-W2.5-H0.9-P0.50-BL_TPS63070RNMR.wrl"
+		(model "${KIPRJMOD}/lib/lcsc.3dshapes/VQFN-HR-15_L3.0-W2.5-H0.9-P0.50-BL_TPS63070RNMR.step"
 			(offset
 				(xyz -0 0.18 -0)
@@
 					(face "Blender Pro Bold")
 					(size 0.5 0.5)
-					(thickness 0.15)
+					(thickness 0.125)
 				)
 			)
@@
 		)
 		(embedded_fonts no)
-		(model "/hardware/lib/lcsc.3dshapes/IND-SMD_L4.0-W4.0-A.wrl"
+		(model "${KIPRJMOD}/lib/lcsc.3dshapes/IND-SMD_L4.0-W4.0-A.step"
 			(offset
 				(xyz 0 -0 -0)
@@
 					(face "Blender Pro Bold")
 					(size 0.5 0.5)
-					(thickness 0.15)
+					(thickness 0.125)
 				)
 			)
@@
 		)
 		(embedded_fonts no)
-		(model "/hardware/lib/lcsc.3dshapes/L0603_L1.6-W0.8-H0.5_BEAD.wrl"
+		(model "${KIPRJMOD}/lib/lcsc.3dshapes/L0603_L1.6-W0.8-H0.5_BEAD.step"
 			(offset
-				(xyz 1.66 -0.49 -0)
+				(xyz 0 0 -0)
 			)
 			(scale
@@
 			)
 			(rotate
-				(xyz 0 0 180)
+				(xyz -0 -0 180)
 			)
 		)
@@
 		)
 		(embedded_fonts no)
-		(model "/hardware/lib/lcsc.3dshapes/SW-SMD_L3.9-W2.9-H2.0-LS4.8.wrl"
+		(model "${KIPRJMOD}/lib/lcsc.3dshapes/SW-SMD_L3.9-W2.9-H2.0-LS4.8.step"
 			(offset
 				(xyz 0 -0 -0)
@@
 					(face "Blender Pro Bold")
 					(size 0.5 0.5)
-					(thickness 0.15)
+					(thickness 0.125)
 				)
 			)
@@
 		)
 		(embedded_fonts no)
-		(model "/hardware/lib/lcsc.3dshapes/L2520.wrl"
+		(model "${KIPRJMOD}/lib/lcsc.3dshapes/L2520.step"
 			(offset
 				(xyz 0 -0 -0)
@@
 					(face "Blender Pro Bold")
 					(size 0.5 0.5)
-					(thickness 0.15)
+					(thickness 0.125)
 				)
 			)
@@
 		)
 		(embedded_fonts no)
-		(model "/hardware/lib/lcsc.3dshapes/FC-135R_L3.2-W1.5.wrl"
+		(model "${KIPRJMOD}/lib/lcsc.3dshapes/FC-135R_L3.2-W1.5.step"
 			(offset
 				(xyz 0 -0 -0)
@@
 					(face "Blender Pro Bold")
 					(size 0.5 0.5)
-					(thickness 0.15)
+					(thickness 0.125)
 				)
 			)
@@
 		)
 		(embedded_fonts no)
-		(model "/hardware/lib/lcsc.3dshapes/TF-SMD_TF-01A.wrl"
+		(model "${KIPRJMOD}/lib/lcsc.3dshapes/TF-SMD_TF-01A.step"
 			(offset
-				(xyz 0 -2.18 0.6)
+				(xyz 0 -5 0)
 			)
 			(scale
@@
 			)
 			(rotate
-				(xyz 0 0 0)
+				(xyz -0 -0 -0)
 			)
 		)
@@
 		)
 		(embedded_fonts no)
-		(model "/hardware/lib/lcsc.3dshapes/SW-SMD_L3.9-W2.9-H2.0-LS4.8.wrl"
+		(model "${KIPRJMOD}/lib/lcsc.3dshapes/SW-SMD_L3.9-W2.9-H2.0-LS4.8.step"
 			(offset
 				(xyz 0 -0 -0)
@@
 		(net 3)
 	)
+	(via
+		(at 149.7 126.55)
+		(size 0.6)
+		(drill 0.3)
+		(layers "F.Cu" "B.Cu")
+		(free yes)
+		(net 3)
+	)
+	(via
+		(at 161.45 112.8)
+		(size 0.6)
+		(drill 0.3)
+		(layers "F.Cu" "B.Cu")
+		(free yes)
+		(net 3)
+	)

Commit message: start blender render and hc flag
Parts:
- renumbered D1 to RDY
