File: hardware/SimpleFlightController.kicad_sch (KiCad schematic)
At the start: 79 parts, among them J1 Screw_Terminal_01x02, J2 Conn_01x03, J3 Conn_01x03, SW1 TS-1088-AR02016, SW2 TS-1088-AR02016, U1 BQ25883RGER, U2 ICM-45686, U3 STM32F722RETx, U4 BMP580, U5 TPS63070RNMR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

Commit message: fixstuff
Connections:
- net +3.3V: now also R14.2
- net at C15.2, L7.1, U6.2 (SW): no longer R14.2
Other:
- moved on the sheet: L7, R14, R15
Changed lines of the file:
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@@
 	)
 	(junction
-		(at 234.95 267.97)
-		(diameter 0)
-		(color 0 0 0 0)
-	)
-	(junction
 		(at 49.53 254)
 		(diameter 0)
@@
 	)
 	(junction
+		(at 251.46 267.97)
+		(diameter 0)
+		(color 0 0 0 0)
+	)
+	(junction
 		(at 134.62 48.26)
 		(diameter 0)
@@
 	)
 	(junction
+		(at 251.46 260.35)
+		(diameter 0)
+		(color 0 0 0 0)
+	)
+	(junction
 		(at 224.79 41.91)
 		(diameter 0)
@@
 	)
 	(junction
-		(at 234.95 260.35)
-		(diameter 0)
-		(color 0 0 0 0)
-	)
-	(junction
 		(at 342.9 107.95)
 		(diameter 0)
@@
 	(wire
 		(pts
-			(xy 234.95 275.59) (xy 255.27 275.59)
+			(xy 251.46 275.59) (xy 255.27 275.59)
 		)
 		(stroke
@@
 	(wire
 		(pts
-			(xy 234.95 260.35) (xy 241.3 260.35)
-		)
-		(stroke
-			(width 0)
-			(type default)
-		)
-	)
-	(wire
-		(pts
 			(xy 63.5 175.26) (xy 62.23 175.26)
 		)
@@
 	(wire
 		(pts
-			(xy 227.33 267.97) (xy 234.95 267.97)
+			(xy 227.33 267.97) (xy 251.46 267.97)
 		)
 		(stroke
@@
 	(wire
 		(pts
+			(xy 247.65 260.35) (xy 251.46 260.35)
+		)
+		(stroke
+			(width 0)
+			(type default)
+		)
+	)
+	(wire
+		(pts
 			(xy 39.37 254) (xy 49.53 254)
 		)
@@
 	(wire
 		(pts
-			(xy 231.14 260.35) (xy 234.95 260.35)
+			(xy 231.14 260.35) (xy 237.49 260.35)
 		)
 		(stroke
@@
 	(symbol
 		(lib_id "Device:R")
-		(at 234.95 271.78 180)
+		(at 251.46 271.78 0)
+		(mirror x)
 		(unit 1)
 		(exclude_from_sim no)
@@
 		(dnp no)
 		(property "Reference" "R15"
-			(at 238.76 270.256 0)
+			(at 247.65 270.256 0)
 			(effects
 				(font
@@
 		)
 		(property "Value" "22.1K"
-			(at 239.522 272.542 0)
+			(at 246.888 272.542 0)
 			(effects
 				(font
@@
 		)
 		(property "Footprint" "Resistor_SMD:R_0402_1005Metric"
-			(at 236.728 271.78 90)
+			(at 249.682 271.78 90)
 			(effects
 				(font
@@
 		)
 		(property "Datasheet" "~"
-			(at 234.95 271.78 0)
+			(at 251.46 271.78 0)
 			(effects
 				(font
@@
 		)
 		(property "Description" "Resistor"
-			(at 234.95 271.78 0)
+			(at 251.46 271.78 0)
 			(effects
 				(font
@@
 		(on_board yes)
 		(dnp no)
-		(fields_autoplaced yes)
 		(property "Reference" "C15"
 			(at 234.95 255.2699 0)
@@
 		)
 		(property "Value" "100nF"
-			(at 234.95 257.8099 0)
+			(at 233.934 257.81 0)
 			(effects
 				(font
@@
 	(symbol
 		(lib_id "Device:R")
-		(at 234.95 264.16 180)
+		(at 251.46 264.16 0)
+		(mirror x)
 		(unit 1)
 		(exclude_from_sim no)
@@
 		(dnp no)
 		(property "Reference" "R14"
-			(at 238.76 262.636 0)
+			(at 247.65 262.636 0)
 			(effects
 				(font
@@
 		)
 		(property "Value" "100K"
-			(at 239.268 264.922 0)
+			(at 247.142 264.922 0)
 			(effects
 				(font
@@
 		)
 		(property "Footprint" "Resistor_SMD:R_0402_1005Metric"
-			(at 236.728 264.16 90)
+			(at 249.682 264.16 90)
 			(effects
 				(font
@@
 		)
 		(property "Datasheet" "~"
-			(at 234.95 264.16 0)
+			(at 251.46 264.16 0)
 			(effects
 				(font
@@
 		)
 		(property "Description" "Resistor"
-			(at 234.95 264.16 0)
+			(at 251.46 264.16 0)
 			(effects
 				(font
@@
 	(symbol
 		(lib_id "lcsc:YHNR3015-5R6M")
-		(at 246.38 260.35 0)
+		(at 242.57 260.35 0)
 		(unit 1)
 		(exclude_from_sim no)
@@
 		(dnp no)
 		(property "Reference" "L7"
-			(at 246.38 254 0)
+			(at 242.57 255.27 0)
 			(effects
 				(font
@@
 		)
 		(property "Value" "YHNR3015-5R6M"
-			(at 251.206 257.556 0)
+			(at 249.428 257.556 0)
 			(effects
 				(font
@@
 		)
 		(property "Footprint" "lcsc:IND-SMD_L3.0-W3.0"
-			(at 246.38 267.97 0)
+			(at 242.57 267.97 0)
 			(effects
 				(font
@@
 		)
 		(property "Datasheet" ""
-			(at 246.38 260.35 0)
+			(at 242.57 260.35 0)
 			(effects
 				(font
@@
 		)
 		(property "Description" ""
-			(at 246.38 260.35 0)
+			(at 242.57 260.35 0)
 			(effects
 				(font
@@
 		)
 		(property "LCSC Part" "C18236327"
-			(at 246.38 270.51 0)
+			(at 242.57 270.51 0)
 			(effects
 				(font
